File: lab4/lab4 task2.kicad_pcb (KiCad board)
At the start: 2 copper layers, 33 x 31.8 mm, 10 parts, among them J1 +9V, U1 NE555D

Commit message: Added gerber files
Parts:
- moved J1 2.54 mm to (157.5, 81.3)
Routing:
- net +9V: track 40.3 -> 50.1 mm
- net GND: track 58.9 -> 64.8 mm
Other:
- board size 33 x 31.8 mm -> 29.2 x 34.3 mm
